Commit message: [models] Add model config files, export path in package.xml

File: models/car/urdf/rusted_car.urdf.xacro (robot description, xacro)
@@ -14,5 +14,5 @@
         <origin xyz="0 0 0" rpy="0 0 0" />
         <geometry>
-           <mesh filename="package://frontier_exploration_3d/models/car/meshes/car_mesh_1500.dae"
+           <mesh filename="package://uav_frontier_exploration_3d/models/car/meshes/car_mesh_1500.dae"
             scale="0.6 0.6 0.6" />
         </geometry>
@@ -21,5 +21,5 @@
         <origin xyz="0 0 0" rpy="0 0 0"/>
         <geometry>
-           <mesh filename="package://frontier_exploration_3d/models/car/meshes/car_mesh_1500.dae"
+           <mesh filename="package://uav_frontier_exploration_3d/models/car/meshes/car_mesh_1500.dae"
             scale="0.6 0.6 0.6" />
         </geometry>

File: models/container/urdf/container.urdf.xacro (robot description, xacro)
@@ -14,5 +14,5 @@
         <origin xyz="0 0 0" rpy="0 0 0" />
         <geometry>
-           <mesh filename="package://frontier_exploration_3d/models/container/meshes/container_mesh_1000.dae"
+           <mesh filename="package://uav_frontier_exploration_3d/models/container/meshes/container_mesh_1000.dae"
             scale="5 5 4" />
         </geometry>
@@ -21,5 +21,5 @@
         <origin xyz="0 0 0" rpy="0 0 0"/>
         <geometry>
-           <mesh filename="package://frontier_exploration_3d/models/container/meshes/container_mesh_1000.dae"
+           <mesh filename="package://uav_frontier_exploration_3d/models/container/meshes/container_mesh_1000.dae"
             scale="5 5 4" />
         </geometry>

File: models/old_building/urdf/old_building.urdf.xacro (robot description, xacro)
@@ -14,5 +14,5 @@
         <origin xyz="0 0 0" rpy="0 0 0" />
         <geometry>
-           <mesh filename="package://frontier_exploration_3d/models/old_building/meshes/building.dae"
+           <mesh filename="package://uav_frontier_exploration_3d/models/old_building/meshes/building.dae"
             scale="15 8 4" />
         </geometry>
@@ -21,5 +21,5 @@
         <origin xyz="0 0 0" rpy="0 0 0"/>
         <geometry>
-           <mesh filename="package://frontier_exploration_3d/models/old_building/meshes/building.dae"
+           <mesh filename="package://uav_frontier_exploration_3d/models/old_building/meshes/building.dae"
             scale="15 8 4" />
         </geometry>

File: models/tower/urdf/mbzirc_tower.urdf.xacro (robot description, xacro)
@@ -15,5 +15,5 @@
         <origin xyz="0 0 0" rpy="0 0 -1.57" />
         <geometry>
-          <mesh filename="package://frontier_exploration_3d/models/tower/meshes/mbzirc_Tower.dae"
+          <mesh filename="package://uav_frontier_exploration_3d/models/tower/meshes/mbzirc_Tower.dae"
             scale="1 1 1" />
         </geometry>
@@ -22,5 +22,5 @@
         <origin xyz="0 0 0" rpy="0 0 -1.57"/>
         <geometry>
-          <mesh filename="package://frontier_exploration_3d/models/tower/meshes/mbzirc_Tower.dae"
+          <mesh filename="package://uav_frontier_exploration_3d/models/tower/meshes/mbzirc_Tower.dae"
             scale="1 1 1" />
         </geometry>

File: models/tower/urdf/tower.urdf.xacro (robot description, xacro)
@@ -14,5 +14,5 @@
         <origin xyz="0 0 0" rpy="0 0 0" />
         <geometry>
-           <mesh filename="package://frontier_exploration_3d/models/tower/meshes/tower.dae"
+           <mesh filename="package://uav_frontier_exploration_3d/models/tower/meshes/tower.dae"
             scale="1 1 1" />
         </geometry>
@@ -21,5 +21,5 @@
         <origin xyz="0 0 0" rpy="0 0 0"/>
         <geometry>
-           <mesh filename="package://frontier_exploration_3d/models/tower/meshes/tower.dae"
+           <mesh filename="package://uav_frontier_exploration_3d/models/tower/meshes/tower.dae"
             scale="1 1 1" />
         </geometry>

File: models/tree/urdf/tree.urdf.xacro (robot description, xacro)
@@ -15,5 +15,5 @@
         <origin xyz="0 0 0" rpy="0 0 0" />
         <geometry>
-          <mesh filename="package://frontier_exploration_3d/models/tree/meshes/tree_25k_mesh.dae" scale="0.4 0.4 0.6" />
+          <mesh filename="package://uav_frontier_exploration_3d/models/tree/meshes/tree_25k_mesh.dae" scale="0.4 0.4 0.6" />
         </geometry>
       </visual>
@@ -21,5 +21,5 @@
         <origin xyz="0 0 0" rpy="0 0 0"/>
         <geometry>
-          <mesh filename="package://frontier_exploration_3d/models/tree/meshes/tree_25k_mesh.dae" scale="0.4 0.4 0.6" />
+          <mesh filename="package://uav_frontier_exploration_3d/models/tree/meshes/tree_25k_mesh.dae" scale="0.4 0.4 0.6" />
         </geometry>
       </collision>
